File: UccMicroDuino/UccMicroDuino.kicad_pcb (KiCad board)
At the start: 2 copper layers, 8 parts, among them J1 Conn_01x10_Socket, J2 USB_A, U1 ATtiny85-20S

Commit message: Add files via upload
Parts:
- added R2: 68Ω 5% 1/8W, Resistor_SMD:R_0805_2012Metric_Pad1.20x1.40mm_HandSolder, F.Cu at (1.88, 0.97)
- added R3: 330Ω 5% 1/8W, Resistor_SMD:R_0805_2012Metric_Pad1.20x1.40mm_HandSolder, F.Cu at (1.88, 3.92)
- added R4: 330Ω 5% 1/8W, Resistor_SMD:R_0805_2012Metric_Pad1.20x1.40mm_HandSolder, F.Cu at (1.88, 6.88)
- C1: value C -> 0.1u
- D1: value D_Filled -> PMLL4148L; footprint Diode_SMD:D_MiniMELF -> Diode_SMD:D_MicroMELF_Handsoldering
- D2: value D_Zener -> 3.6V 1/2mW; footprint Diode_SMD:D_SOD-123 -> Diode_SMD:D_MicroMELF_Handsoldering
- D3: value LED -> 3.6V 1/2mW; footprint ledSmd:ledSMD -> Diode_SMD:D_MicroMELF_Handsoldering
- J2: value USB_A -> Conn_01x10_Socket; footprint embeddedPcbUsb:USB_A_UCC -> Connector_PinHeader_2.54mm:PinHeader_1x10_P2.54mm_Vertical
- R1: value R -> 1.5KΩ 5% 1/8W
Connections:
- C1 pad 1: unconnected-(C1-Pad1) -> +5V
- C1 pad 2: unconnected-(C1-Pad2) -> GND
- D1 pad 2: unconnected-(D1-A-Pad2) -> Net-(D1-A)
- D2 pad 1: unconnected-(D2-K-Pad1) -> Net-(D2-K)
- D2 pad 2: unconnected-(D2-A-Pad2) -> GND
- D3 pad 1: unconnected-(D3-K-Pad1) -> Net-(D3-K)
- D3 pad 2: unconnected-(D3-A-Pad2) -> GND
- J2 pad 1: unconnected-(J2-VBUS-Pad1) -> +5V
- J2 pad 2: unconnected-(J2-D--Pad2) -> GND
- J2 pad 4: unconnected-(J2-GND-Pad4) -> Net-(J2-Pin_4)
- R1 pad 2: unconnected-(R1-Pad2) -> Net-(D2-K)
- U1 pad 1: unconnected-(U1-~{RESET}/PB5-Pad1) -> Net-(J2-Pin_9)
- U1 pad 2: unconnected-(U1-XTAL1/PB3-Pad2) -> Net-(J2-Pin_7)
- U1 pad 3: unconnected-(U1-XTAL2/PB4-Pad3) -> Net-(J2-Pin_8)
- U1 pad 4: unconnected-(U1-GND-Pad4) -> GND
- U1 pad 5: unconnected-(U1-AREF/PB0-Pad5) -> Net-(J2-Pin_4)
- U1 pad 6: unconnected-(U1-PB1-Pad6) -> Net-(D4-A)
- U1 pad 7: unconnected-(U1-PB2-Pad7) -> Net-(J2-Pin_6)
- U1 pad 8: unconnected-(U1-VCC-Pad8) -> +5V
Other:
- board outline added: 57 x 54 mm
